Commit message: feat: Update LIDAR configuration and launch file for improved integration

File: src/minibot/description/lidar.xacro (robot description, xacro)
@@ -3,5 +3,6 @@
     <xacro:property name="lidar_radius"             value="0.025"/>
     <xacro:property name="lidar_thickness"          value="0.040"/>
-    <xacro:property name="lidar_offset_x"           value="0.230"/>
+    <!-- Centrado en X respecto al link 'chasis' -->
+    <xacro:property name="lidar_offset_x"           value="${chassis_length/2}"/>
     <xacro:property name="lidar_offset_z"           value="0.098"/>
     <!-- Lidar -->
@@ -62,8 +63,7 @@
                 </noise>
             </lidar>
-        <plugin filename="gz-sim-sensors-system"
-                name="gz::sim::systems::Sensors">
+            <plugin filename="gz-sim-sensors-system" name="gz::sim::systems::Sensors">
                 <render_engine>ogre2</render_engine>
-        </plugin>
+            </plugin>
         </sensor>
     </gazebo>

File: src/minibot/description/robot_main.xacro (robot description, xacro)
@@ -1,69 +1,57 @@
 <?xml version="1.0"?>
 <robot xmlns:xacro="http://www.ros.org/wiki/xacro">
-    <xacro:include filename = "inertial_macros.xacro" />
-    <xacro:property name="chassis_length"           value="0.320"/>
-    <xacro:property name="chassis_width"            value="0.240"/>
-    <xacro:property name="chassis_height"           value="0.078"/>
-    <xacro:property name="chassis_mass"             value="0.700"/>
-    <xacro:property name="wheel_radius"             value="0.034"/>
-    <xacro:property name="wheel_thickness"          value="0.026"/>
-    <xacro:property name="wheel_mass"               value="0.050"/>
-    <xacro:property name="wheel_offset_x"           value="0.133"/>
-    <xacro:property name="wheel_offset_y"           value="0.133"/>
-    <xacro:property name="wheel_offset_z"           value="0.020"/>
-    <xacro:property name="caster_wheel_radius"      value="${wheel_radius - wheel_offset_z}"/>
-    <xacro:property name="caster_wheel_mass"        value="0.010"/>
-    <xacro:property name="caster_wheel_offset_x"    value="0.230"/>
-    <xacro:property name="caster_wheel_offset_z"    value="${wheel_offset_z - wheel_radius + caster_wheel_radius}"/>
-    <!-- Colors -->
-    <material name="white">
-        <color rgba= "1 1 1 1"/>
-    </material>
-    <material name="black">
-        <color rgba= "0 0 0 1"/>
-    </material>
-    <material name= "orange">
-        <color rgba= "1 0.25 0 1"/>
-    </material>
-    <material name="cyan">
-        <color rgba= "0 1 1 1"/>
-    </material>
-    <material name="indigo">
-        <color rgba= "0.294 0 0.51 1"/>
-    </material>
-    <!-- convention (except base_link): joint followed by link -->
-    <!-- base_link -->
-    <link name="base_link">
-    </link>
-    <!-- base_footprint -->
+    <xacro:include filename="inertial_macros.xacro"/>
+    <!-- Dimensiones del chasis -->
+    <xacro:property name="chassis_length"  value="0.320"/>
+    <xacro:property name="chassis_width"   value="0.240"/>
+    <xacro:property name="chassis_height"  value="0.078"/>
+    <xacro:property name="chassis_mass"    value="0.700"/>
+    <!-- Ruedas -->
+    <xacro:property name="wheel_radius"    value="0.034"/>
+    <xacro:property name="wheel_thickness" value="0.026"/>
+    <xacro:property name="wheel_mass"      value="0.050"/>
+    <!-- Geometría: vía y altura de rueda (se mantiene la que traías) -->
+    <xacro:property name="wheel_offset_y"  value="0.133"/>  <!-- mitad del ancho de vía -->
+    <xacro:property name="wheel_offset_z"  value="0.020"/>
+    <!-- Nueva distancia entre ejes (Ackermann) -->
+    <xacro:property name="wheelbase"       value="${chassis_length}"/><!-- eje trasero en x=0, eje delantero en x=0.20 -->
+    <!-- Materiales -->
+    <material name="white"><color rgba="1 1 1 1"/></material>
+    <material name="black"><color rgba="0 0 0 1"/></material>
+    <material name="orange"><color rgba="1 0.25 0 1"/></material>
+    <material name="cyan"><color rgba="0 1 1 1"/></material>
+    <material name="indigo"><color rgba="0.294 0 0.51 1"/></material>
+    <!-- base_link y base_footprint -->
+    <link name="base_link"/>
     <joint name="base_footprint_joint" type="fixed">
-        <parent link= "base_link"/>
-        <child link= "base_footprint"/>
-        <origin xyz= "0 0 0" rpy= "0 0 0"/>
+        <parent link="base_link"/>
+        <child link="base_footprint"/>
+        <origin xyz="0 0 0" rpy="0 0 0"/>
     </joint>
-    <link name="base_footprint">
-    </link>
-    <!-- chasis -->
+    <link name="base_footprint"/>
+    <!-- Chasis (coincide con tu convención de nombre 'chasis') -->
+    <!-- Lo ubicamos igual que antes: su centro queda en (chassis_length/2, 0, chassis_height/2) -->
     <joint name="chasis_joint" type="fixed">
-        <parent link= "base_link"/>
-        <child link= "chasis"/>
-        <origin xyz= "${-wheel_offset_x} 0 ${-wheel_offset_z}"/>
+        <parent link="base_link"/>
+        <child link="chasis"/>
+        <origin xyz="0 0 ${-wheel_offset_z}"/>
     </joint>
     <link name="chasis">
         <visual>
-            <origin xyz= "${chassis_length/2} 0 ${chassis_height/2}" rpy= "0 0 0"/>
+            <origin xyz="${chassis_length/2} 0 ${chassis_height/2}"/>
             <geometry>
-                <box size = "${chassis_length} ${chassis_width} ${chassis_height}"/>
+                <box size="${chassis_length} ${chassis_width} ${chassis_height}"/>
             </geometry>
-            <material name= "black"/>
+            <material name="black"/>
         </visual>
         <collision>
-            <origin xyz= "${chassis_length/2} 0 ${chassis_height/2}" rpy= "0 0 0"/>
+            <origin xyz="${chassis_length/2} 0 ${chassis_height/2}"/>
             <geometry>
-                <box size = "${chassis_length} ${chassis_width} ${chassis_height}"/>
+                <box size="${chassis_length} ${chassis_width} ${chassis_height}"/>
             </geometry>
         </collision>
-        <xacro:inertial_box mass= "0.5" x="${chassis_length}" y="${chassis_width}" z="${chassis_height}">
-            <origin xyz= "${chassis_length/2} 0 ${chassis_height/2}" rpy= "0 0 0"/>
+        <xacro:inertial_box mass="${chassis_mass}"
+                            x="${chassis_length}" y="${chassis_width}" z="${chassis_height}">
+            <origin xyz="${chassis_length/2} 0 ${chassis_height/2}"/>
         </xacro:inertial_box>
     </link>
@@ -71,82 +59,141 @@
         <material>Gazebo/Black</material>
     </gazebo>
-    <!-- left_wheel -->
-    <joint name="left_wheel_joint" type="continuous">
-        <parent link= "base_link"/>
-        <child link= "left_wheel"/>
-        <origin xyz= "0 ${wheel_offset_y} 0" rpy = "${pi/2} 0 0"/>
-        <axis xyz= "0 0 -1"/>
+    <!-- ======================= EJE TRASERO (x = 0) ======================= -->
+    <joint name="rear_left_wheel_joint" type="continuous">
+        <parent link="base_link"/>
+        <child  link="rear_left_wheel"/>
+        <origin xyz="0 ${wheel_offset_y} 0" rpy="${pi/2} 0 0"/>
+        <axis xyz="0 0 -1"/>
     </joint>
-    <link name="left_wheel">
+    <link name="rear_left_wheel">
         <visual>
             <geometry>
-                <cylinder radius = "${wheel_radius}" length= "${wheel_thickness}"/>
+                <cylinder radius="${wheel_radius}" length="${wheel_thickness}"/>
             </geometry>
-            <material name= "orange"/>
+            <material name="orange"/>
         </visual>
         <collision>
-            <geometry>
-                <sphere radius = "${wheel_radius}" />
-            </geometry>
+            <geometry><sphere radius="${wheel_radius}"/></geometry>
         </collision>
-        <xacro:inertial_cylinder mass = "${wheel_mass}" radius= "${wheel_radius}" length= "${wheel_thickness}">
-            <origin xyz= "0 0 0" rpy= "0 0 0"/>
+        <xacro:inertial_cylinder mass="${wheel_mass}"
+                                 radius="${wheel_radius}" length="${wheel_thickness}">
+            <origin xyz="0 0 0"/>
         </xacro:inertial_cylinder>
     </link>
-    <gazebo reference="left_wheel">
+    <gazebo reference="rear_left_wheel">
         <material>Gazebo/Orange</material>
     </gazebo>
-    <!-- right_wheel -->
-    <joint name="right_wheel_joint" type="continuous">
-        <parent link= "base_link"/>
-        <child link= "right_wheel"/>
-        <origin xyz= "0 ${-wheel_offset_y} 0" rpy = "${pi/2} 0 0"/>
-        <axis xyz= "0 0 -1"/>
+    <joint name="rear_right_wheel_joint" type="continuous">
+        <parent link="base_link"/>
+        <child  link="rear_right_wheel"/>
+        <origin xyz="0 ${-wheel_offset_y} 0" rpy="${pi/2} 0 0"/>
+        <axis xyz="0 0 -1"/>
     </joint>
-    <link name="right_wheel">
+    <link name="rear_right_wheel">
         <visual>
             <geometry>
-                <cylinder radius = "${wheel_radius}" length= "${wheel_thickness}"/>
+                <cylinder radius="${wheel_radius}" length="${wheel_thickness}"/>
             </geometry>
-            <material name= "orange"/>
+            <material name="orange"/>
         </visual>
         <collision>
-            <geometry>
-                <sphere radius = "${wheel_radius}" />
-            </geometry>
+            <geometry><sphere radius="${wheel_radius}"/></geometry>
         </collision>
-        <xacro:inertial_cylinder mass = "${wheel_mass}" radius= "${wheel_radius}" length= "${wheel_thickness}">
-            <origin xyz= "0 0 0" rpy= "0 0 0"/>
+        <xacro:inertial_cylinder mass="${wheel_mass}"
+                                 radius="${wheel_radius}" length="${wheel_thickness}">
+            <origin xyz="0 0 0"/>
         </xacro:inertial_cylinder>
     </link>
-    <gazebo reference="right_wheel">
+    <gazebo reference="rear_right_wheel">
         <material>Gazebo/Orange</material>
     </gazebo>
-    <!-- caster_wheel -->
-    <joint name="caster_wheel_joint" type="fixed">
-        <parent link= "chasis"/>
-        <child link= "caster_wheel"/>
-        <origin xyz= "${caster_wheel_offset_x} 0 0"/>
+    <!-- ======================= EJE DELANTERO (x = wheelbase) ======================= -->
+    <!-- Articulación de dirección (mangueta) izquierda -->
+    <joint name="front_left_steer_joint" type="revolute">
+        <parent link="base_link"/>
+        <child  link="front_left_steer"/>
+        <origin xyz="${wheelbase} ${wheel_offset_y} 0"/>
+        <axis xyz="0 0 1"/>
+        <limit effort="5.0" velocity="2.0" lower="-0.6" upper="0.6"/>
     </joint>
-    <link name="caster_wheel">
+    <link name="front_left_steer">
+        <visual>
+            <origin xyz="0 0 0"/>
+            <geometry><sphere radius="0.01"/></geometry>
+            <material name="cyan"/>
+        </visual>
+        <collision><geometry><sphere radius="0.01"/></geometry></collision>
+        <xacro:inertial_sphere mass="0.01" radius="0.01">
+            <origin xyz="0 0 0"/>
+        </xacro:inertial_sphere>
+    </link>
+    <!-- Rueda delantera izquierda bajo la mangueta -->
+    <joint name="front_left_wheel_joint" type="continuous">
+        <parent link="front_left_steer"/>
+        <child  link="front_left_wheel"/>
+        <origin xyz="0 0 0" rpy="${pi/2} 0 0"/>
+        <axis xyz="0 0 -1"/>
+    </joint>
+    <link name="front_left_wheel">
         <visual>
             <geometry>
-                <sphere radius = "${caster_wheel_radius}"/>
+                <cylinder radius="${wheel_radius}" length="${wheel_thickness}"/>
             </geometry>
-            <material name= "orange"/>
+            <material name="orange"/>
         </visual>
         <collision>
-            <geometry>
-                <sphere radius = "${caster_wheel_radius}"/>
-            </geometry>
+            <geometry><sphere radius="${wheel_radius}"/></geometry>
         </collision>
-        <xacro:inertial_sphere mass= "${caster_wheel_mass}" radius= "${caster_wheel_radius}">
-            <origin xyz= "0 0 0" rpy= "0 0 0"/>
+        <xacro:inertial_cylinder mass="${wheel_mass}"
+                                 radius="${wheel_radius}" length="${wheel_thickness}">
+            <origin xyz="0 0 0"/>
+        </xacro:inertial_cylinder>
+    </link>
+    <gazebo reference="front_left_wheel">
+        <material>Gazebo/Orange</material>
+    </gazebo>
+    <!-- Articulación de dirección (mangueta) derecha -->
+    <joint name="front_right_steer_joint" type="revolute">
+        <parent link="base_link"/>
+        <child  link="front_right_steer"/>
+        <origin xyz="${wheelbase} ${-wheel_offset_y} 0"/>
+        <axis xyz="0 0 1"/>
+        <limit effort="5.0" velocity="2.0" lower="-0.6" upper="0.6"/>
+    </joint>
+    <link name="front_right_steer">
+        <visual>
+            <origin xyz="0 0 0"/>
+            <geometry><sphere radius="0.01"/></geometry>
+            <material name="cyan"/>
+        </visual>
+        <collision><geometry><sphere radius="0.01"/></geometry></collision>
+        <xacro:inertial_sphere mass="0.01" radius="0.01">
+            <origin xyz="0 0 0"/>
         </xacro:inertial_sphere>
     </link>
-    <gazebo reference="caster_wheel">
+    <!-- Rueda delantera derecha bajo la mangueta -->
+    <joint name="front_right_wheel_joint" type="continuous">
+        <parent link="front_right_steer"/>
+        <child  link="front_right_wheel"/>
+        <origin xyz="0 0 0" rpy="${pi/2} 0 0"/>
+        <axis xyz="0 0 -1"/>
+    </joint>
+    <link name="front_right_wheel">
+        <visual>
+            <geometry>
+                <cylinder radius="${wheel_radius}" length="${wheel_thickness}"/>
+            </geometry>
+            <material name="orange"/>
+        </visual>
+        <collision>
+            <geometry><sphere radius="${wheel_radius}"/></geometry>
+        </collision>
+        <xacro:inertial_cylinder mass="${wheel_mass}"
+                                 radius="${wheel_radius}" length="${wheel_thickness}">
+            <origin xyz="0 0 0"/>
+        </xacro:inertial_cylinder>
+    </link>
+    <gazebo reference="front_right_wheel">
         <material>Gazebo/Orange</material>
-        <mu1 value= "0.0001"/>
-        <mu2 value= "0.0001"/>
     </gazebo>
 </robot>

Commit message: feat: Update launch files and world configuration for improved simulation environment

File: src/minibot/description/lidar.xacro (robot description, xacro)
@@ -3,8 +3,6 @@
     <xacro:property name="lidar_radius"             value="0.025"/>
     <xacro:property name="lidar_thickness"          value="0.040"/>
-    <!-- Centrado en X respecto al link 'chasis' -->
     <xacro:property name="lidar_offset_x"           value="${chassis_length/2}"/>
     <xacro:property name="lidar_offset_z"           value="0.098"/>
-    <!-- Lidar -->
     <joint name="lidar_joint" type="fixed">
         <parent link="chasis"/>
@@ -28,5 +26,4 @@
         </xacro:inertial_cylinder>
     </link>
-    <!-- Lidar in gazebo-->
     <gazebo reference="lidar_frame">
         <sensor name="lidar" type="gpu_lidar">
@@ -63,8 +60,5 @@
                 </noise>
             </lidar>
-            <plugin filename="gz-sim-sensors-system" name="gz::sim::systems::Sensors">
-                <render_engine>ogre2</render_engine>
-            </plugin>
-        </sensor>
+            </sensor>
     </gazebo>
 </robot>

File: src/minibot/description/robot_main.xacro (robot description, xacro)
@@ -2,19 +2,14 @@
 <robot xmlns:xacro="http://www.ros.org/wiki/xacro">
     <xacro:include filename="inertial_macros.xacro"/>
-    <!-- Dimensiones del chasis -->
     <xacro:property name="chassis_length"  value="0.320"/>
     <xacro:property name="chassis_width"   value="0.240"/>
     <xacro:property name="chassis_height"  value="0.078"/>
     <xacro:property name="chassis_mass"    value="0.700"/>
-    <!-- Ruedas -->
     <xacro:property name="wheel_radius"    value="0.034"/>
     <xacro:property name="wheel_thickness" value="0.026"/>
     <xacro:property name="wheel_mass"      value="0.050"/>
-    <!-- Geometría: vía y altura de rueda (se mantiene la que traías) -->
-    <xacro:property name="wheel_offset_y"  value="0.133"/>  <!-- mitad del ancho de vía -->
+    <xacro:property name="wheel_offset_y"  value="0.133"/>
     <xacro:property name="wheel_offset_z"  value="0.020"/>
-    <!-- Nueva distancia entre ejes (Ackermann) -->
-    <xacro:property name="wheelbase"       value="${chassis_length}"/><!-- eje trasero en x=0, eje delantero en x=0.20 -->
-    <!-- Materiales -->
+    <xacro:property name="wheelbase"       value="${chassis_length}"/>
     <material name="white"><color rgba="1 1 1 1"/></material>
     <material name="black"><color rgba="0 0 0 1"/></material>
@@ -22,5 +17,4 @@
     <material name="cyan"><color rgba="0 1 1 1"/></material>
     <material name="indigo"><color rgba="0.294 0 0.51 1"/></material>
-    <!-- base_link y base_footprint -->
     <link name="base_link"/>
     <joint name="base_footprint_joint" type="fixed">
@@ -30,6 +24,4 @@
     </joint>
     <link name="base_footprint"/>
-    <!-- Chasis (coincide con tu convención de nombre 'chasis') -->
-    <!-- Lo ubicamos igual que antes: su centro queda en (chassis_length/2, 0, chassis_height/2) -->
     <joint name="chasis_joint" type="fixed">
         <parent link="base_link"/>
@@ -56,8 +48,4 @@
         </xacro:inertial_box>
     </link>
-    <gazebo reference="chasis">
-        <material>Gazebo/Black</material>
-    </gazebo>
-    <!-- ======================= EJE TRASERO (x = 0) ======================= -->
     <joint name="rear_left_wheel_joint" type="continuous">
         <parent link="base_link"/>
@@ -81,7 +69,4 @@
         </xacro:inertial_cylinder>
     </link>
-    <gazebo reference="rear_left_wheel">
-        <material>Gazebo/Orange</material>
-    </gazebo>
     <joint name="rear_right_wheel_joint" type="continuous">
         <parent link="base_link"/>
@@ -105,9 +90,4 @@
         </xacro:inertial_cylinder>
     </link>
-    <gazebo reference="rear_right_wheel">
-        <material>Gazebo/Orange</material>
-    </gazebo>
-    <!-- ======================= EJE DELANTERO (x = wheelbase) ======================= -->
-    <!-- Articulación de dirección (mangueta) izquierda -->
     <joint name="front_left_steer_joint" type="revolute">
         <parent link="base_link"/>
@@ -128,5 +108,4 @@
         </xacro:inertial_sphere>
     </link>
-    <!-- Rueda delantera izquierda bajo la mangueta -->
     <joint name="front_left_wheel_joint" type="continuous">
         <parent link="front_left_steer"/>
@@ -150,8 +129,4 @@
         </xacro:inertial_cylinder>
     </link>
-    <gazebo reference="front_left_wheel">
-        <material>Gazebo/Orange</material>
-    </gazebo>
-    <!-- Articulación de dirección (mangueta) derecha -->
     <joint name="front_right_steer_joint" type="revolute">
         <parent link="base_link"/>
@@ -172,5 +147,4 @@
         </xacro:inertial_sphere>
     </link>
-    <!-- Rueda delantera derecha bajo la mangueta -->
     <joint name="front_right_wheel_joint" type="continuous">
         <parent link="front_right_steer"/>
@@ -194,7 +168,4 @@
         </xacro:inertial_cylinder>
     </link>
-    <gazebo reference="front_right_wheel">
-        <material>Gazebo/Orange</material>
-    </gazebo>
     <gazebo>
         <plugin filename="gz-sim-ackermann-steering-system" name="gz::sim::systems::AckermannSteering">
@@ -212,8 +183,10 @@
             <min_acceleration>-3</min_acceleration>
             <max_acceleration>3</max_acceleration>
-            <topic>/cmd_vel</topic> </plugin>
+            <topic>/cmd_vel</topic>
+        </plugin>
         <plugin filename="gz-sim-odometry-publisher-system" name="gz::sim::systems::OdometryPublisher">
             <odom_frame>odom</odom_frame>
-            <robot_base_frame>base_link</robot_base_frame> <odom_publish_frequency>50</odom_publish_frequency>
+            <robot_base_frame>base_link</robot_base_frame>
+            <odom_publish_frequency>50</odom_publish_frequency>
             <topic>/odom</topic>
             <tf_topic>/tf</tf_topic>
